Commit message: Finished adding PhantomX measurements and STLs

File: src/hexapod_description/urdf/hexapod_model_phantomx.xacro (robot description, xacro)
@@ -3,9 +3,9 @@
 	<!-- parameters -->
 	<xacro:property name="pi" value="3.1415926535897931" />
-	<xacro:property name="body_length_x" value="0.3556" />
-	<xacro:property name="body_length_y" value="0.165" />
-	<xacro:property name="coxa_length" value="0.05893" />
-	<xacro:property name="femur_length" value="0.10798" />
-	<xacro:property name="tibia_length" value="0.08774" />
+	<xacro:property name="body_length_x" value="0.250" />
+	<xacro:property name="body_length_y" value="0.125" />
+	<xacro:property name="coxa_length" value="0.052" />
+	<xacro:property name="femur_length" value="0.065" />
+	<xacro:property name="tibia_length" value="0.133" />
 	<!-- Build the body frame -->
     <link name="footprint" />
@@ -112,9 +112,9 @@
 	</xacro:macro>
 <!-- Build robot model -->
-	<xacro:leg side="R" position="R" x="-0.1778" y="-0.0825" angle="-${pi*3/4}" axis="1" />
-	<xacro:leg side="R" position="M" x="0.0" y="-0.13335" angle="-${pi/2}" axis="1" />
-	<xacro:leg side="R" position="F" x="0.1778" y="-0.0825" angle="-${pi/4}" axis="1" />
-	<xacro:leg side="L" position="R" x="-0.1778" y="0.0825" angle="${pi*3/4}" axis="-1" />
-	<xacro:leg side="L" position="M" x="0.0" y="0.13335" angle="${pi/2}" axis="-1" />
-	<xacro:leg side="L" position="F" x="0.1778" y="0.0825" angle="${pi/4}" axis="-1" />
+	<xacro:leg side="R" position="R" x="-0.120" y="-0.060" angle="-${pi*3/4}" axis="1" />
+	<xacro:leg side="R" position="M" x="0.0" y="-0.100" angle="-${pi/2}" axis="1" />
+	<xacro:leg side="R" position="F" x="0.120" y="-0.060" angle="-${pi/4}" axis="1" />
+	<xacro:leg side="L" position="R" x="-0.120" y="0.060" angle="${pi*3/4}" axis="-1" />
+	<xacro:leg side="L" position="M" x="0.0" y="0.100" angle="${pi/2}" axis="-1" />
+	<xacro:leg side="L" position="F" x="0.120" y="0.060" angle="${pi/4}" axis="-1" />
 </robot>

Commit message: Syncing with Master

File: src/hexapod_description/urdf/hexapod_model_phantomx.xacro (robot description, xacro)
@@ -8,9 +8,8 @@
 	<xacro:property name="femur_length" value="0.065" />
 	<xacro:property name="tibia_length" value="0.133" />
-	<!-- Build the body frame -->
-    <link name="footprint" />
-    <joint name="footprint_joint" type="fixed">
-        <parent link="footprint"/>
-        <child link="base_link"/>
+	<link name="base_footprint" />
+		<joint name="footprint_joint" type="fixed">
+		<parent link="base_footprint"/>
+		<child link="base_link"/>
 		<origin xyz="0 0 0" rpy="0 0 0" />
     </joint>
@@ -18,8 +17,8 @@
 	<joint name="base_joint" type="fixed">
 		<parent link="base_link" />
-		<child link="body" />
+		<child link="body_link" />
 		<origin xyz="0 0 0" rpy="0 0 0" />
 	</joint>
-	<link name="body">
+	<link name="body_link">
 			<visual>
 	  			<origin	xyz="0 0 0" rpy="0 0 0" />
@@ -32,11 +31,22 @@
 			</visual>
 	</link>
-	<joint name="camera" type="fixed">
-		<parent link="base_link" />
-		<child link="camera_link" />
-		<origin xyz="0 0 0" rpy="${pi/2} ${pi} ${pi/2}" />
+	<joint name="camera_rgb_joint" type="fixed">
+		<parent link="body_link" />
+		<child link="camera_rgb_link" />
+		<origin xyz="0.150 0.0255 0.034" rpy="${pi/2} ${pi} ${pi/2}" />
 	</joint>
-	<link name="camera_link">
-	</link>
+	<link name="camera_rgb_link" />
+	<joint name="camera_depth_joint" type="fixed">
+		<parent link="body_link" />
+		<child link="camera_depth_link" />
+		<origin xyz="0.135 0.065 0.080" rpy="${pi/2} ${pi} ${pi/2}" />
+	</joint>
+	<link name="camera_depth_link" />
+	<joint name="imu_joint" type="fixed">
+		<parent link="base_footprint" />
+		<child link="imu_link" />
+		<origin xyz="0 0 0" rpy="${pi} 0 0" />
+	</joint>
+	<link name="imu_link" />
 	<!-- Joint properties -->
 	<xacro:property name="joint_lower_limit" value="-${3.14}" />
@@ -49,5 +59,5 @@
 		<joint name="leg_center_joint_${side}${position}" type="fixed">
 			<origin xyz="${x} ${y} 0" rpy="0 0 0" />
-			<parent link="body" />
+			<parent link="body_link" />
 			<child link="leg_center_${side}${position}" />
 		</joint>

Commit message: Setup IMU for CH Robotics UM7; Adjust math odom scaling;

File: src/hexapod_description/urdf/hexapod_model_phantomx.xacro (robot description, xacro)
@@ -9,5 +9,5 @@
 	<xacro:property name="tibia_length" value="0.133" />
 	<link name="base_footprint" />
-		<joint name="footprint_joint" type="fixed">
+	<joint name="footprint_joint" type="fixed">
 		<parent link="base_footprint"/>
 		<child link="base_link"/>
@@ -46,5 +46,5 @@
 		<parent link="base_footprint" />
 		<child link="imu_link" />
-		<origin xyz="0 0 0" rpy="${pi} 0 0" />
+		<origin xyz="0 0 0" rpy="0 0 0" />
 	</joint>
 	<link name="imu_link" />

Commit message: More pan and tilt scanner functionality

File: src/hexapod_description/urdf/hexapod_model_phantomx.xacro (robot description, xacro)
@@ -31,16 +31,38 @@
 			</visual>
 	</link>
+	<joint name="head_pan_joint" type="revolute">
+		<parent link="body_link"/>
+		<child link="head_pan_link"/>
+		<axis xyz="0 0 1" />
+		<origin xyz="0.145 0.0 0.080" />
+		<limit lower="-${3.14}" upper="${3.14}" effort="10000" velocity="100" />
+	</joint>
+	<link name="head_pan_link"/>
+	<joint name="head_tilt_joint" type="revolute">
+		<parent link="head_pan_link"/>
+		<child link="head_tilt_link"/>
+		<axis xyz="0 1 0" />
+		<origin xyz="0.0 0.0 0.020" />
+		<limit lower="-${3.14}" upper="${3.14}" effort="10000" velocity="100" />
+	</joint>
+	<link name="head_tilt_link"/>
 	<joint name="camera_rgb_joint" type="fixed">
-		<parent link="body_link" />
+		<parent link="head_tilt_link" />
 		<child link="camera_rgb_link" />
-		<origin xyz="0.150 0.0255 0.034" rpy="${pi/2} ${pi} ${pi/2}" />
+		<origin xyz="0.0 0.0 0.0" rpy="${pi/2} ${pi} ${pi/2}" />
 	</joint>
 	<link name="camera_rgb_link" />
 	<joint name="camera_depth_joint" type="fixed">
-		<parent link="body_link" />
+		<parent link="head_tilt_link" />
 		<child link="camera_depth_link" />
-		<origin xyz="0.135 0.065 0.080" rpy="${pi/2} ${pi} ${pi/2}" />
+		<origin xyz="0.0 0.0 0.0" rpy="${pi/2} ${pi} ${pi/2}" />
 	</joint>
 	<link name="camera_depth_link" />
+<joint name="camera_depth_frame" type="fixed">
+	<parent link="head_tilt_link" />
+	<child link="camera_depth_frame_link" />
+	<origin xyz="0.0 0.0 0.0" />
+</joint>
+<link name="camera_depth_frame_link" />
 	<joint name="imu_joint" type="fixed">
 		<parent link="base_footprint" />

Commit message: Sync with master: 1cb75dc: localization tweaks and refinements.

File: src/hexapod_description/urdf/hexapod_model_phantomx.xacro (robot description, xacro)
@@ -1,3 +1,3 @@
-<?xml version="1.0"?>
+<?xml version="1.0" encoding="UTF-8" ?>
 <robot xmlns:xacro="http://ros.org/wiki/xacro" name="PhantomX">
 	<!-- parameters -->
@@ -8,16 +8,10 @@
 	<xacro:property name="femur_length" value="0.065" />
 	<xacro:property name="tibia_length" value="0.133" />
-	<link name="base_footprint" />
-	<joint name="footprint_joint" type="fixed">
-		<parent link="base_footprint"/>
-		<child link="base_link"/>
-		<origin xyz="0 0 0" rpy="0 0 0" />
+	<link name="base_link" />
+    <joint name="base_joint" type="fixed">
+        <parent link="base_link" />
+        <child link="body_link" />
+        <origin xyz="0 0 0" rpy="0 0 0" />
     </joint>
-	<link name="base_link" />
-	<joint name="base_joint" type="fixed">
-		<parent link="base_link" />
-		<child link="body_link" />
-		<origin xyz="0 0 0" rpy="0 0 0" />
-	</joint>
 	<link name="body_link">
 			<visual>
@@ -31,4 +25,5 @@
 			</visual>
 	</link>
+	<!-- Head Pan and Tilt properties -->
 	<joint name="head_pan_joint" type="revolute">
 		<parent link="body_link"/>
@@ -47,16 +42,17 @@
 	</joint>
 	<link name="head_tilt_link"/>
+	<!-- Camera properties -->
 	<joint name="camera_rgb_joint" type="fixed">
 		<parent link="head_tilt_link" />
-		<child link="camera_rgb_link" />
+		<child link="camera_rgb_optical_frame" />
 		<origin xyz="0.0 0.0 0.0" rpy="${pi/2} ${pi} ${pi/2}" />
 	</joint>
-	<link name="camera_rgb_link" />
+	<link name="camera_rgb_optical_frame" />
 	<joint name="camera_depth_joint" type="fixed">
 		<parent link="head_tilt_link" />
-		<child link="camera_depth_link" />
+		<child link="camera_depth_optical_frame" />
 		<origin xyz="0.0 0.0 0.0" rpy="${pi/2} ${pi} ${pi/2}" />
 	</joint>
-	<link name="camera_depth_link" />
+	<link name="camera_depth_optical_frame" />
 <joint name="camera_depth_frame" type="fixed">
 	<parent link="head_tilt_link" />
@@ -65,6 +61,7 @@
 </joint>
 <link name="camera_depth_frame_link" />
+	<!-- IMU properties -->
 	<joint name="imu_joint" type="fixed">
-		<parent link="base_footprint" />
+		<parent link="base_link" />
 		<child link="imu_link" />
 		<origin xyz="0 0 0" rpy="0 0 0" />

Commit message: Syncing with master.

File: src/hexapod_description/urdf/hexapod_model_phantomx.xacro (robot description, xacro)
@@ -12,9 +12,9 @@
         <parent link="base_link" />
         <child link="body_link" />
-        <origin xyz="0 0 0" rpy="0 0 0" />
+        <origin xyz="0.0 0.0 0.0" rpy="0.0 0.0 0.0" />
     </joint>
 	<link name="body_link">
 			<visual>
-	  			<origin	xyz="0 0 0" rpy="0 0 0" />
+	  			<origin	xyz="0.0 0.0 0.0" rpy="0.0 0.0 0.0" />
       			<geometry>
         			<mesh filename="package://hexapod_description/meshes/body_phantomx.stl" scale="0.001 0.001 0.001"/>
@@ -29,5 +29,5 @@
 		<parent link="body_link"/>
 		<child link="head_pan_link"/>
-		<axis xyz="0 0 1" />
+		<axis xyz="0.0 0.0 1.0" />
 		<origin xyz="0.145 0.0 0.080" />
 		<limit lower="-${3.14}" upper="${3.14}" effort="10000" velocity="100" />
@@ -37,5 +37,5 @@
 		<parent link="head_pan_link"/>
 		<child link="head_tilt_link"/>
-		<axis xyz="0 1 0" />
+		<axis xyz="0.0 1.0 0.0" />
 		<origin xyz="0.0 0.0 0.020" />
 		<limit lower="-${3.14}" upper="${3.14}" effort="10000" velocity="100" />
@@ -65,5 +65,5 @@
 		<parent link="base_link" />
 		<child link="imu_link" />
-		<origin xyz="0 0 0" rpy="0 0 0" />
+		<origin xyz="0.0 0.0 0.0" rpy="0.0 0.0 0.0" />
 	</joint>
 	<link name="imu_link" />
@@ -77,5 +77,5 @@
 		<!-- leg position -->
 		<joint name="leg_center_joint_${side}${position}" type="fixed">
-			<origin xyz="${x} ${y} 0" rpy="0 0 0" />
+			<origin xyz="${x} ${y} 0.0" rpy="0.0 0.0 0.0" />
 			<parent link="body_link" />
 			<child link="leg_center_${side}${position}" />
@@ -84,13 +84,13 @@
 		<!-- coxa -->
 		<joint name="coxa_joint_${side}${position}" type="revolute">
-			<origin xyz="0 0 0" rpy="0 0 ${angle}" />
+			<origin xyz="0.0 0.0 0.0" rpy="0.0 0.0 ${angle}" />
 			<parent link="leg_center_${side}${position}" />
 			<child link="coxa_${side}${position}" />
-			<axis xyz="0 0 ${-axis}" />
+			<axis xyz="0.0 0.0 ${-axis}" />
 			<limit lower="${joint_lower_limit}" upper="${joint_upper_limit}" effort="${joint_effort}" velocity="${joint_velocity}" />
 		</joint>
 		<link name="coxa_${side}${position}">
 			<visual>
-				<origin xyz="0 0 0" rpy="0 0 0" />
+				<origin xyz="0.0 0.0 0.0" rpy="0.0 0.0 0.0" />
       			<geometry>
         			<mesh filename="package://hexapod_description/meshes/coxa_phantomx.stl" scale="0.001 0.001 0.001"/>
@@ -103,13 +103,13 @@
 		<!-- femur -->
 		<joint name="femur_joint_${side}${position}" type="revolute">
-			<origin xyz="${coxa_length} 0 0" rpy="-${pi/2} 0 0" />
+			<origin xyz="${coxa_length} 0.0 0.0" rpy="-${pi/2} 0.0 0.0" />
 			<parent link="coxa_${side}${position}" />
 			<child link="femur_${side}${position}" />
-			<axis xyz="0 0 ${axis}" />
+			<axis xyz="0.0 0.0 ${axis}" />
 			<limit lower="${joint_lower_limit}" upper="${joint_upper_limit}" effort="${joint_effort}" velocity="${joint_velocity}" />
 		</joint>
 		<link name="femur_${side}${position}">
 			<visual>
-				<origin xyz="0 0 0" rpy="0 0 0" />
+				<origin xyz="0.0 0.0 0.0" rpy="0.0 0.0 0.0" />
       			<geometry>
         			<mesh filename="package://hexapod_description/meshes/femur_phantomx.stl" scale="0.001 0.001 0.001"/>
@@ -122,13 +122,13 @@
 		<!-- tibia -->
 		<joint name="tibia_joint_${side}${position}" type="revolute">
-			<origin xyz="0 -${femur_length} 0" rpy="${pi} 0 0" />
+			<origin xyz="0.0 -${femur_length} 0.0" rpy="${pi} 0.0 0.0" />
 			<parent link="femur_${side}${position}" />
 			<child link="tibia_${side}${position}" />
-			<axis xyz="0 0 ${axis}" />
+			<axis xyz="0.0 0.0 ${axis}" />
 			<limit lower="${joint_lower_limit}" upper="${joint_upper_limit}" effort="${joint_effort}" velocity="${joint_velocity}" />
 		</joint>
 		<link name="tibia_${side}${position}">
 			<visual>
-				<origin xyz="0 0 0" rpy="0 0 0" />
+				<origin xyz="0.0 0.0 0.0" rpy="0.0 0.0 0.0" />
       			<geometry>
         			<mesh filename="package://hexapod_description/meshes/tibia_phantomx.stl" scale="0.001 0.001 0.001"/>
